File: Pico_Debug_Stack.kicad_pcb (KiCad board)
At the start: 4 copper layers, 43 x 98 mm, 146 parts, among them J1 Stack to Motherboard Connector, J10 USB_A, J2 Scope_TP, J3 BM03B-SRSS-TB, J4 Conn_01x04_Pin, J7 Conn_01x04, J8 Scope_TP_21-40, SW2 Tactile Button, 160gf, SW3 Tactile Button, 160gf, SW4 Tactile Button, 160gf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

Commit message: Added holes for USB C socket
Made this v0.1.2
Routing:
- net GND: track 1751.9 -> 1751.2 mm, vias 84 -> 91
Changed lines of the file:
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@@
 	)
 	(via
+		(at 111.07 116.17)
+		(size 0.6)
+		(drill 0.3)
+		(layers "F.Cu" "B.Cu")
+		(free yes)
+		(net 3)
+	)
+	(via
 		(at 121.58 136.545)
 		(size 0.6)
@@
 	)
 	(via
+		(at 112.37 75.3)
+		(size 0.6)
+		(drill 0.3)
+		(layers "F.Cu" "B.Cu")
+		(free yes)
+		(net 3)
+	)
+	(via
 		(at 119.21 71.79)
 		(size 0.6)
@@
 	)
 	(via
+		(at 107.3 75.52)
+		(size 0.6)
+		(drill 0.3)
+		(layers "F.Cu" "B.Cu")
+		(free yes)
+		(net 3)
+	)
+	(via
 		(at 97.06 137.42)
 		(size 0.6)
@@
 	)
 	(via
+		(at 122.63 82.93)
+		(size 0.6)
+		(drill 0.3)
+		(layers "F.Cu" "B.Cu")
+		(free yes)
+		(net 3)
+	)
+	(via
 		(at 115.9965 122.17)
 		(size 0.6)
@@
 	)
 	(via
+		(at 109.16 118.83)
+		(size 0.6)
+		(drill 0.3)
+		(layers "F.Cu" "B.Cu")
+		(free yes)
+		(net 3)
+	)
+	(via
 		(at 126.42 138.0135)
 		(size 0.6)
@@
 	)
 	(via
+		(at 115.81 156.15)
+		(size 0.6)
+		(drill 0.3)
+		(layers "F.Cu" "B.Cu")
+		(free yes)
+		(net 3)
+	)
+	(via
 		(at 117.29 91.21)
 		(size 0.6)
@@
 	)
 	(via
+		(at 99.74 156.32)
+		(size 0.6)
+		(drill 0.3)
+		(layers "F.Cu" "B.Cu")
+		(free yes)
+		(net 3)
+	)
+	(via
 		(at 91.25 85.18)
 		(size 0.6)
@@
 	)
 	(segment
-		(start 105.539373 90.75)
-		(end 105.539373 90.509373)
-		(width 0.127)
-		(layer "In1.Cu")
-		(net 3)
-	)
-	(segment
 		(start 106.307543 88.912457)
 		(end 106.38 88.84)
@@
 		(width 0.127)
 		(layer "In1.Cu")
-		(net 3)
-	)
-	(segment
-		(start 105.539373 90.509373)
-		(end 105.2 90.17)
-		(width 0.127)
-		(layer "In1.Cu")
