File: Pico_Debug_Stack.kicad_sch (KiCad schematic)
At the start: 146 parts, among them J1 Stack to Motherboard Connector, J10 USB_A, J2 Scope_TP, J3 BM03B-SRSS-TB, J4 Conn_01x04_Pin, J7 Conn_01x04, J8 Scope_TP_21-40, SW2 Tactile Button, 160gf, SW3 Tactile Button, 160gf, SW4 Tactile Button, 160gf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

Commit message: Replace wrong version with Version 0.1.1
Parts:
- J1: now fitted
- J10: JLCPCB C112455 -> (none); LCSC (none) -> C112455
Connections:
- net GND: now also C6.2
- net at C6.1: now also R28.2, U3.13 (RESET)
Other:
- moved on the sheet: C6

Commit message: note about USB C cables
Other:
- note added: "Do not buy 4 wire USB C cables for this. You must use four wire USB A cables, or you won't git power to pass through."
